File: Electronics/Front_left_lamp/Front_left_lamp_v1.brd (EAGLE design)
At the start: 42.9 x 26.7 mm, 9 parts

Commit message: Front lamps done
Parts:
- R4: value 1K -> 680
Changed lines of the file:
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@@
 <element name="R2" library="resistor" package="0204V" value="4K7" x="19.05" y="12.7" rot="R270"/>
 <element name="R3" library="resistor" package="0204V" value="4K7" x="33.02" y="12.7" rot="R270"/>
-<element name="R4" library="resistor" package="0204V" value="1K" x="26.67" y="6.35" rot="R180"/>
+<element name="R4" library="resistor" package="0204V" value="680" x="26.67" y="6.35" rot="R180"/>
 </elements>
 <signals>
