File: Electronics/Rear_left_lamp/Rear_left_lamp_v1.brd (EAGLE design)
At the start: 58.1 x 14 mm, 11 parts, among them X1 JST-XH-05-PIN-ROUND-PAD

Commit message: Rear lamps improved
Greater resistors' value for API_START_ENGINE
Parts:
- R1, R2: value 3K3 -> 6K8
Changed lines of the file:
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@@
 <attribute name="CURRENT" value="0.14 mA" x="54.61" y="3.81" size="1.778" layer="27" display="off"/>
 </element>
-<element name="R1" library="resistor" package="0204V" value="3K3" x="29.21" y="10.16" rot="R90"/>
-<element name="R2" library="resistor" package="0204V" value="3K3" x="21.59" y="10.16" rot="R90"/>
+<element name="R1" library="resistor" package="0204V" value="6K8" x="29.21" y="10.16" rot="R90"/>
+<element name="R2" library="resistor" package="0204V" value="6K8" x="21.59" y="10.16" rot="R90"/>
 <element name="R3" library="resistor" package="0204V" value="680" x="5.08" y="10.16" rot="R90"/>
 <element name="R4" library="resistor" package="0204V" value="1K" x="12.7" y="10.16" rot="R90"/>
