File: Electronics/Regular/Front_left_lamp/Front_left_lamp_v5.brd (EAGLE design)
At the start: 29.2 x 12.7 mm, 7 parts, among them X2 JST-XH-03-PIN-LONG-PAD

Commit message: BOM on front lamps added
Parts:
- LED1, LED2, LED3: value 2.58 V -> White
- LED4: value 1.88 V -> Yellow
- moved R2 0.90 mm to (20.3, 7.62)
Routing:
- net N$2: track 3.71 -> 4.61 mm
- net API_TURN_LEFT: track 10.2 -> 9.32 mm
