File: Electronics/Regular/Front_right_lamp/Front_right_lamp_v5.brd (EAGLE design)
At the start: 29.2 x 12.7 mm, 7 parts, among them X2 JST-XH-03-PIN-LONG-PAD

Commit message: BOM on front lamps added
Parts:
- LED1, LED2, LED3: value 2.58 V -> White
- LED4: value 1.88 V -> Yellow
- moved LED1 15.2 mm to (12.7, 2.54)
- moved LED3 15.2 mm to (27.9, 2.54)
