File: Electronics/Regular/Rear_brake_lamp/Rear_brake_lamp_v4.brd (EAGLE design)
At the start: 48.3 x 8.9 mm, 8 parts, among them X2 JST-XH-02-PIN-LONG-PAD

Commit message: BOM on all the lamps added
Note: Version of lamps' projects has increased from x.0 to x.1.

What also has been done:
- some visual refactoring on schematics
Parts:
- LED1, LED2, LED3, LED4, LED5, LED6: value 1.78 V -> Red
- R1: value 120 -> 150
