File: Electronics/Regular/Rear_right_lamp/Rear_right_lamp_v4.brd (EAGLE design)
At the start: 50.8 x 12.7 mm, 10 parts, among them X2 JST-XH-05-PIN-LONG-PAD

Commit message: BOM on all the lamps added
Note: Version of lamps' projects has increased from x.0 to x.1.

What also has been done:
- some visual refactoring on schematics
Parts:
- LED1, LED2, LED4: value 1.83 V -> Red
- LED3: value 1.88 V -> Yellow
- LED5: value 2.58 V -> White
