File: Electronics/Lamp_dispatcher/Lamp_dispatcher.sch (EAGLE design)
At the start: 6 parts, among them X1 JST-XH-06-PIN-LONG-PAD, X2 JST-XH-02-PIN-LONG-PAD, X3 JST-XH-03-PIN-LONG-PAD, X4 JST-XH-03-PIN-LONG-PAD, X5 JST-XH-05-PIN-LONG-PAD, X6 JST-XH-05-PIN-LONG-PAD

Commit message: Lamp dispatcher improved
What has been improved:
- rotated 2- and 6-pin JST connectors,
- corrected PCB dimensions,
- curved GND wire
Connections:
- net API_BRAKE: now also X1-3.S, X2-2.S; no longer X1-4.S, X2-1.S
- net API_START_ENGINE: now also X1-6.S; no longer X1-1.S
- net API_TURN_LEFT: now also X1-5.S; no longer X1-2.S
- net API_TURN_RIGHT: now also X1-4.S; no longer X1-3.S
- net API_WITHDRAW: now also X1-2.S; no longer X1-5.S
- net GND: now also X1-1.S, X2-1.S; no longer X1-6.S, X2-2.S
Other:
- note added: "1.1"
- note removed: "1.0"
- moved on the sheet: X1-1, X1-2, X1-3, X1-4, X1-5, X1-6, X2-1, X2-2, X3-1, X3-2, X3-3, X4-1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
