File: Electronics/Fuse_protector/Fuse_protector.sch (EAGLE design)
At the start: 12 parts

Commit message: Fuse protector improved
What has been improved:
- corrected size of space for fuses
Other:
- note added: "1.1"
- note removed: "1.0"
Changed lines of the file:
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@@
 <text x="175.26" y="27.94" size="2.54" layer="94">Author: sesame0707</text>
 <text x="205.994" y="11.43" size="2.54" layer="94">9</text>
-<text x="261.62" y="7.112" size="2.54" layer="94">1.0</text>
+<text x="261.62" y="7.112" size="2.54" layer="94">1.1</text>
 </plain>
 <instances>
